Commit message: modified model

File: dualarm_mod.urdf (robot description, URDF)
Before this commit: robot dualarm, 16 links, 15 joints
Joints:
- joint j0: origin xyz=0 0.159800001842985 0.9227 rpy=1.5707963267949 0 1.57079632679488 -> xyz=0 0.159800001842985 0.5727 rpy=1.5707963267949 0 1.57079632679488

Commit message: modified model

File: dualarm_mod.urdf (robot description, URDF)
Before this commit: robot dualarm, 16 links, 15 joints
Joints:
- joint j1: axis 0 0 1 -> 0 0 -1
- joint j8: axis 0 0 -1 -> 0 0 1
